Commit message: Can stand up but tremble.

File: inverted_pendulum_description/urdf/inverted_pendulum.xacro (robot description, xacro)
@@ -1,80 +1,84 @@
 <?xml version="1.0" ?>
-<robot name="inverted_pendulum" xmlns:xacro="http://www.ros.org/wiki/xacro">
-<xacro:include filename="$(find inverted_pendulum_description)/urdf/materials.xacro" />
-<xacro:include filename="$(find inverted_pendulum_description)/urdf/inverted_pendulum.trans" />
-<xacro:include filename="$(find inverted_pendulum_description)/urdf/inverted_pendulum.gazebo" />
-<link name="base_link">
-  <inertial>
-    <origin xyz="0.0 0.05 0.0" rpy="0 0 0"/>
-    <mass value="1.8368"/>
-    <inertia ixx="0.005357" iyy="0.010044" izz="0.006605" ixy="0.0" iyz="0" ixz="0.0"/>
-  </inertial>
-  <visual>
-    <origin xyz="0 0 0" rpy="0 0 0"/>
-    <geometry>
-      <mesh filename="package://inverted_pendulum_description/meshes/base_link.stl" scale="0.001 0.001 0.001"/>
-    </geometry>
-    <material name="silver"/>
-  </visual>
-  <collision>
-    <origin xyz="0 0 0" rpy="0 0 0"/>
-    <geometry>
-      <mesh filename="package://inverted_pendulum_description/meshes/base_link.stl" scale="0.001 0.001 0.001"/>
-    </geometry>
-  </collision>
-</link>
-<link name="leg_1_1">
-  <inertial>
-    <origin xyz="-0.01675 -0.0015 -0.02393" rpy="0 0 0"/>
-    <mass value="0.00208"/>
-    <inertia ixx="1e-06" iyy="1e-06" izz="2.13e-07" ixy="0.0" iyz="0.0" ixz="0.0"/>
-  </inertial>
-  <visual>
-    <origin xyz="-0.018516 -0.0111 -0.141337" rpy="0 0 0"/>
-    <geometry>
-      <mesh filename="package://inverted_pendulum_description/meshes/leg_1_1.stl" scale="0.001 0.001 0.001"/>
-    </geometry>
-    <material name="silver"/>
-  </visual>
-  <collision>
-    <origin xyz="-0.018516 -0.0111 -0.141337" rpy="0 0 0"/>
-    <geometry>
-      <mesh filename="package://inverted_pendulum_description/meshes/leg_1_1.stl" scale="0.001 0.001 0.001"/>
-    </geometry>
-  </collision>
-</link>
-<link name="leg_2_1">
-  <inertial>
-    <origin xyz="0 -0.0015 -0.029" rpy="0 0 0"/>
-    <mass value="0.00208"/>
-    <inertia ixx="1e-06" iyy="1e-06" izz="1.92e-07" ixy="0.0" iyz="0.0" ixz="0.0"/>
-  </inertial>
-  <visual>
-    <origin xyz="0.0146 -0.0081 -0.093" rpy="0 0 0"/>
-    <geometry>
-      <mesh filename="package://inverted_pendulum_description/meshes/leg_2_1.stl" scale="0.001 0.001 0.001"/>
-    </geometry>
-    <material name="silver"/>
-  </visual>
-  <collision>
-    <origin xyz="0.0146 -0.0081 -0.093" rpy="0 0 0"/>
-    <geometry>
-      <mesh filename="package://inverted_pendulum_description/meshes/leg_2_1.stl" scale="0.001 0.001 0.001"/>
-    </geometry>
-  </collision>
-</link>
-<joint name="joint_1" type="revolute">
-  <origin xyz="0.0185 0.0111 0.1413" rpy="0 0 0"/>
-  <parent link="base_link"/>
-  <child link="leg_1_1"/>
-  <axis xyz="0.0 1.0 0.0"/>
-  <limit effort="1.2" velocity="31" lower="-1e10" upper="1e10"/>
-</joint>
-<joint name="joint_2" type="revolute">
-  <origin xyz="-0.033 -0.003 -0.0482" rpy="0 0 0"/>
-  <parent link="leg_1_1"/>
-  <child link="leg_2_1"/>
-  <axis xyz="0.0 1.0 0.0"/>
-  <limit effort="1.2" velocity="31" lower="-1e10" upper="1e10"/>
-</joint>
+<robot xmlns:xacro="http://www.ros.org/wiki/xacro" name="inverted_pendulum">
+    <xacro:include filename="$(find inverted_pendulum_description)/urdf/materials.xacro"/>
+    <xacro:include filename="$(find inverted_pendulum_description)/urdf/inverted_pendulum.trans"/>
+    <xacro:include filename="$(find inverted_pendulum_description)/urdf/inverted_pendulum.gazebo"/>
+    <link name="base_link">
+        <inertial>
+            <origin xyz="0.0 0.05 0.0" rpy="0 0 0"/>
+            <mass value="1.8368"/>
+            <inertia ixx="0.005357" iyy="0.010044" izz="0.006605" ixy="0.0" iyz="0" ixz="0.0"/>
+        </inertial>
+        <visual>
+            <origin xyz="0 0 0" rpy="0 0 0"/>
+            <geometry>
+                <mesh filename="package://inverted_pendulum_description/meshes/base_link.stl"
+                      scale="0.001 0.001 0.001"/>
+            </geometry>
+            <material name="silver"/>
+        </visual>
+        <collision>
+            <origin xyz="0 0 0" rpy="0 0 0"/>
+            <geometry>
+                <mesh filename="package://inverted_pendulum_description/meshes/base_link.stl"
+                      scale="0.001 0.001 0.001"/>
+            </geometry>
+        </collision>
+    </link>
+    <link name="leg_1_1">
+        <inertial>
+            <origin xyz="-0.01675 -0.0015 -0.02393" rpy="0 0 0"/>
+            <mass value="0.00208"/>
+            <inertia ixx="1e-06" iyy="1e-06" izz="2.13e-07" ixy="0.0" iyz="0.0" ixz="0.0"/>
+        </inertial>
+        <visual>
+            <origin xyz="-0.018516 -0.0111 -0.141337" rpy="0 0 0"/>
+            <geometry>
+                <mesh filename="package://inverted_pendulum_description/meshes/leg_1_1.stl" scale="0.001 0.001 0.001"/>
+            </geometry>
+            <material name="silver"/>
+        </visual>
+        <collision>
+            <origin xyz="-0.018516 -0.0111 -0.141337" rpy="0 0 0"/>
+            <geometry>
+                <mesh filename="package://inverted_pendulum_description/meshes/leg_1_1.stl" scale="0.001 0.001 0.001"/>
+            </geometry>
+        </collision>
+    </link>
+    <link name="leg_2_1">
+        <inertial>
+            <origin xyz="0 -0.0015 -0.029" rpy="0 0 0"/>
+            <mass value="0.00208"/>
+            <inertia ixx="1e-06" iyy="1e-06" izz="1.92e-07" ixy="0.0" iyz="0.0" ixz="0.0"/>
+        </inertial>
+        <visual>
+            <origin xyz="0.0146 -0.0081 -0.093" rpy="0 0 0"/>
+            <geometry>
+                <mesh filename="package://inverted_pendulum_description/meshes/leg_2_1.stl" scale="0.001 0.001 0.001"/>
+            </geometry>
+            <material name="silver"/>
+        </visual>
+        <collision>
+            <origin xyz="0.0146 -0.0081 -0.093" rpy="0 0 0"/>
+            <geometry>
+                <mesh filename="package://inverted_pendulum_description/meshes/leg_2_1.stl" scale="0.001 0.001 0.001"/>
+            </geometry>
+        </collision>
+    </link>
+    <joint name="joint_1" type="revolute">
+        <origin xyz="0.0185 0.0111 0.1413" rpy="0 0 0"/>
+        <parent link="base_link"/>
+        <child link="leg_1_1"/>
+        <axis xyz="0.0 1.0 0.0"/>
+        <limit effort="0.05" velocity="1" lower="-1e10" upper="1e10"/>
+        <dynamics damping="0" friction="0.0002"/>
+    </joint>
+    <joint name="joint_2" type="revolute">
+        <origin xyz="-0.033 -0.003 -0.0482" rpy="0 0 0"/>
+        <parent link="leg_1_1"/>
+        <child link="leg_2_1"/>
+        <axis xyz="0.0 1.0 0.0"/>
+        <limit effort="0.05" velocity="1" lower="-1e10" upper="1e10"/>
+        <dynamics damping="0" friction="0.0002"/>
+    </joint>
 </robot>

Commit message: Add dynamic config.

File: inverted_pendulum_description/urdf/inverted_pendulum.xacro (robot description, xacro)
@@ -71,5 +71,5 @@
         <child link="leg_1_1"/>
         <axis xyz="0.0 1.0 0.0"/>
-        <limit effort="0.05" velocity="1" lower="-1e10" upper="1e10"/>
+        <limit effort="0.1" velocity="1" lower="-1e10" upper="1e10"/>
         <dynamics damping="0" friction="0.0002"/>
     </joint>
@@ -79,6 +79,6 @@
         <child link="leg_2_1"/>
         <axis xyz="0.0 1.0 0.0"/>
-        <limit effort="0.05" velocity="1" lower="-1e10" upper="1e10"/>
-        <dynamics damping="0" friction="0.0002"/>
+        <limit effort="0.1" velocity="1" lower="-1e10" upper="1e10"/>
+        <dynamics damping="0" friction="0.0001"/>
     </joint>
 </robot>
